Commit message: Sensors added (LIDAR, Camera, IMU)

File: Resources/robots/pioneer.urdf (robot description, URDF)
Before this commit: robot pioneer3at_body, 15 links, 14 joints
Links:
- added link cam_frame; visual box size=0.01 0.05 0.01
- added link cam_optical_link
- added link laser_frame, mass 1e-5; collision box size=0.01 0.01 0.01; visual mesh filename=../meshes/hokuyo1.dae
Joints:
- added joint cam_joint: type fixed, parent chassis, child cam_frame, origin xyz=0.24 0 0.084 rpy=0 0 0
- added joint cam_optical_joint: type fixed, parent cam_frame, child cam_optical_link, origin xyz=0.3 0 0.2 rpy=-1.65 0 -1.65
- added joint laser_joint: type fixed, parent chassis, child laser_frame, origin xyz=0.2 0 0.104 rpy=0 0 0
